Commit message: xacroファイルの修正

File: adrv_description/urdf/adrv.urdf.xacro (robot description, xacro)
@@ -9,5 +9,5 @@
   <link name="base_link">
     <visual>
-      <origin xyz="0 0 0" rpy="0 0 0" />
+      <origin xyz="0 0 0" rpy="0 0 ${M_PI/2}" />
       <geometry>
         <mesh filename="package://adrv_description/meshes/base_link.dae" />
@@ -15,5 +15,5 @@
     </visual>
     <collision>
-      <origin xyz="0 0 0" rpy="0 0 0" />
+      <origin xyz="0 0 0" rpy="0 0 ${M_PI/2}" />
       <geometry>
         <mesh filename="package://adrv_description/meshes/base_link.dae" />
@@ -30,7 +30,10 @@
   <!-- wheel_link -->
   <xacro:include filename="$(find adrv_description)/urdf/wheel.urdf.xacro" />
-  <xacro:wheel name="wheel_FR" pose_xyz="0 0 0" pose_rpy="0 0 0" />
+  <xacro:wheel name="wheel_FR" pose_xyz="0.09 0.075 0.015" pose_rpy="0 0 ${M_PI/2}" />
+  <xacro:wheel name="wheel_FL" pose_xyz="0.09 -0.075 0.015" pose_rpy="0 0 -${M_PI/2}" />
+  <xacro:wheel name="wheel_RR" pose_xyz="-0.09 0.075 0.015" pose_rpy="0 0 ${M_PI/2}" />
+  <xacro:wheel name="wheel_RL" pose_xyz="-0.09 -0.075 0.015" pose_rpy="0 0 -${M_PI/2}" />
   <!-- Gazebo plugins -->
-  <!-- <gazebo>
+  <gazebo>
     <plugin name="gazebo_ros_control" filename="libgazebo_ros_control.so">
       <robotNamespace>/</robotNamespace>
@@ -38,4 +41,4 @@
       <legacyModeNS>true</legacyModeNS>
     </plugin>
-  </gazebo> -->
+  </gazebo>
 </robot>

File: adrv_description/urdf/wheel.urdf.xacro (robot description, xacro)
@@ -6,5 +6,5 @@
         <origin xyz="0 0 0" rpy="0 0 0" />
         <geometry>
-          <mesh filename="package://adrv_description/meshes/wheel.dae" />
+          <mesh filename="package://adrv_description/meshes/wheel_link.dae" />
         </geometry>
       </visual>
@@ -12,5 +12,5 @@
         <origin xyz="0 0 0" rpy="0 0 0" />
         <geometry>
-          <mesh filename="package://adrv_description/meshes/wheel.dae" />
+          <mesh filename="package://adrv_description/meshes/wheel_link.dae" />
         </geometry>
       </collision>
@@ -19,6 +19,6 @@
         <mass value="1.0" />
         <inertia ixx="1.0" ixy="0.0" ixz="0.0"
-                          iyy="1.0" iyz="0.0"
-                                    izz="1.0" />
+                           iyy="1.0" iyz="0.0"
+                                     izz="1.0" />
       </inertial>
     </link>
@@ -34,5 +34,5 @@
       <child link="${name}_link" />
       <origin xyz="${pose_xyz}" rpy="${pose_rpy}" />
-      <axis xyz="0 1 0" rpy="0 0 0" />
+      <axis xyz="1 0 0" rpy="0 0 0" />
     </joint>
     <transmission name="${name}_trans" type="SimpleTransmission">

Commit message: complete robot_description

File: adrv_description/urdf/adrv.urdf.xacro (robot description, xacro)
@@ -9,5 +9,5 @@
   <link name="base_link">
     <visual>
-      <origin xyz="0 0 0" rpy="0 0 ${M_PI/2}" />
+      <origin xyz="0 0 0" rpy="0 0 ${-M_PI/2}" />
       <geometry>
         <mesh filename="package://adrv_description/meshes/base_link.dae" />
@@ -15,5 +15,5 @@
     </visual>
     <collision>
-      <origin xyz="0 0 0" rpy="0 0 ${M_PI/2}" />
+      <origin xyz="0 0 0" rpy="0 0 ${-M_PI/2}" />
       <geometry>
         <mesh filename="package://adrv_description/meshes/base_link.dae" />
@@ -29,15 +29,16 @@
   </link>
   <!-- wheel_link -->
-  <xacro:include filename="$(find adrv_description)/urdf/wheel.urdf.xacro" />
-  <xacro:wheel name="wheel_FR" pose_xyz="0.09 0.075 0.015" pose_rpy="0 0 ${M_PI/2}" />
-  <xacro:wheel name="wheel_FL" pose_xyz="0.09 -0.075 0.015" pose_rpy="0 0 -${M_PI/2}" />
-  <xacro:wheel name="wheel_RR" pose_xyz="-0.09 0.075 0.015" pose_rpy="0 0 ${M_PI/2}" />
-  <xacro:wheel name="wheel_RL" pose_xyz="-0.09 -0.075 0.015" pose_rpy="0 0 -${M_PI/2}" />
+  <xacro:include filename="$(find adrv_description)/urdf/steering.urdf.xacro" />
+  <xacro:front_steer_shaft base="base_link" pose_xyz="0.095 0 0.016" />
+  <xacro:rear_wheel_shaft base="base_link" pose_xyz="-0.09 0 0.016" tread="0.146" radius="0.032" />
+  <xacro:front_wheel name="wheel_fr" base="base_link" pose_xyz="0.095 -0.073 0.016" right_left="right" />
+  <xacro:front_wheel name="wheel_fl" base="base_link" pose_xyz="0.095 0.073 0.016" right_left="left" />
+  <xacro:rear_wheel name="wheel_rr" base="base_link" pose_xyz="-0.09 -0.073 0.016" right_left="right" />
+  <xacro:rear_wheel name="wheel_rl" base="base_link" pose_xyz="-0.09 0.073 0.016" right_left="left" />
   <!-- Gazebo plugins -->
   <gazebo>
     <plugin name="gazebo_ros_control" filename="libgazebo_ros_control.so">
       <robotNamespace>/</robotNamespace>
-      <robotSimType>gazebo_ros_control/DefaultRobotHWSim</robotSimType>
-      <legacyModeNS>true</legacyModeNS>
+      <robotSimType>steer_bot_hardware_gazebo/SteerBotHardwareGazebo</robotSimType>
     </plugin>
   </gazebo>

File: adrv_description/urdf/wheel.urdf.xacro (robot description, xacro)
@@ -1,18 +1,34 @@
 <?xml version="1.0" ?>
 <robot name="wheel" xmlns:xacro="http://ros.org/wiki/xacro">
-  <xacro:macro name="wheel" params="name pose_xyz pose_rpy">
+  <xacro:macro name="wheel" params="name right_left">
     <link name="${name}_link">
-      <visual>
-        <origin xyz="0 0 0" rpy="0 0 0" />
-        <geometry>
-          <mesh filename="package://adrv_description/meshes/wheel_link.dae" />
-        </geometry>
-      </visual>
-      <collision>
-        <origin xyz="0 0 0" rpy="0 0 0" />
-        <geometry>
-          <mesh filename="package://adrv_description/meshes/wheel_link.dae" />
-        </geometry>
-      </collision>
+      <xacro:if value="${right_left =='right'}">
+        <visual>
+          <origin xyz="0 0 0" rpy="0 0 -${M_PI/2}" />
+          <geometry>
+            <mesh filename="package://adrv_description/meshes/wheel_link.dae" />
+          </geometry>
+        </visual>
+        <collision>
+          <origin xyz="0 0 0" rpy="0 0 -${M_PI/2}" />
+          <geometry>
+            <mesh filename="package://adrv_description/meshes/wheel_link.dae" />
+          </geometry>
+        </collision>
+      </xacro:if>
+      <xacro:if value="${right_left =='left'}">
+        <visual>
+          <origin xyz="0 0 0" rpy="0 0 ${M_PI/2}" />
+          <geometry>
+            <mesh filename="package://adrv_description/meshes/wheel_link.dae" />
+          </geometry>
+        </visual>
+        <collision>
+          <origin xyz="0 0 0" rpy="0 0 ${M_PI/2}" />
+          <geometry>
+            <mesh filename="package://adrv_description/meshes/wheel_link.dae" />
+          </geometry>
+        </collision>
+      </xacro:if>
       <inertial>
         <origin xyz="0 0 0" />
@@ -30,19 +46,4 @@
       <fdir1 value="1 0 0" />
     </gazebo>
-    <joint name="${name}_joint" type="continuous">
-      <parent link="base_link" />
-      <child link="${name}_link" />
-      <origin xyz="${pose_xyz}" rpy="${pose_rpy}" />
-      <axis xyz="1 0 0" rpy="0 0 0" />
-    </joint>
-    <transmission name="${name}_trans" type="SimpleTransmission">
-      <type>transmission_interface/SimpleTransmission</type>
-      <actuator name="${name}_motor">
-        <mechanicalReduction>1</mechanicalReduction>
-      </actuator>
-      <joint name="${name}_joint">
-        <hardwareInterface>hardware_interface/VelocityJointInterface</hardwareInterface>
-      </joint>
-    </transmission>
   </xacro:macro>
 </robot>

Commit message: add sensor in robot description

File: adrv_description/urdf/adrv.urdf.xacro (robot description, xacro)
@@ -36,4 +36,12 @@
   <xacro:rear_wheel name="wheel_rr" base="base_link" pose_xyz="-0.09 -0.073 0.016" right_left="right" />
   <xacro:rear_wheel name="wheel_rl" base="base_link" pose_xyz="-0.09 0.073 0.016" right_left="left" />
+  <!-- YDLIDAR X4 -->
+  <xacro:include filename="$(find adrv_description)/urdf/ydlidar_x4.urdf.xacro" />
+  <xacro:ydlidar_x4 name="ydlidar" base="base_link" pose_xyz="0.052 0 0.066" pose_rpy="0 0 ${-M_PI/2-6/180*M_PI}" />
+  <!-- RealSense D435 -->
+  <xacro:include filename="$(find realsense2_description)/urdf/_d435.urdf.xacro" />
+  <xacro:sensor_d435 parent="base_link" use_nominal_extrinsics="true">
+    <origin xyz="0.127 0 0.042" rpy="0 ${5/180*M_PI} 0"/>
+  </xacro:sensor_d435>
   <!-- Gazebo plugins -->
   <gazebo>

Commit message: オドメトリの情報を取得できるよう修正

File: adrv_description/urdf/adrv.urdf.xacro (robot description, xacro)
@@ -10,4 +10,5 @@
   <xacro:include filename="$(find realsense2_description)/urdf/_d435.urdf.xacro" />
   <xacro:include filename="$(find adrv_description)/urdf/sensor.urdf.xacro" />
+  <xacro:include filename="$(find adrv_description)/urdf/inertia.urdf.xacro" />
   <!-- ###  links  ### -->
   <!-- base_link -->
@@ -25,11 +26,5 @@
       </geometry>
     </collision>
-    <inertial>
-      <origin xyz="0 0 0" />
-      <mass value="1.0" />
-      <inertia ixx="1.0" ixy="0.0" ixz="0.0"
-                         iyy="1.0" iyz="0.0"
-                                   izz="1.0" />
-    </inertial>
+    <xacro:box_inertia mass="10.0" w="0.146" h="0.185" d="0.05" />
   </link>
   <!-- wheel_link -->
@@ -47,5 +42,5 @@
   </xacro:sensor_d435>
   <!-- Sensor -->
-  <xacro:imu name="imu" base="base_link" pose_xyz="0.082 0 0.046" pose_rpy="0 ${M_PI} ${-M_PI/2}" />
+  <xacro:imu name="imu" base="base_link" pose_xyz="0.082 0 0.046" pose_rpy="0 0 0" />
   <!-- Gazebo plugins -->
   <gazebo>

File: adrv_description/urdf/sensor.urdf.xacro (robot description, xacro)
@@ -19,5 +19,5 @@
           <bodyName>${name}_link</bodyName>
           <updateRateHZ>100.0</updateRateHZ>
-          <gaussianNoise>0.0</gaussianNoise>
+          <gaussianNoise>0.001</gaussianNoise>
           <xyzOffset>0 0 0</xyzOffset>
           <rpyOffset>0 0 0</rpyOffset>

File: adrv_description/urdf/steering.urdf.xacro (robot description, xacro)
@@ -64,5 +64,5 @@
       <child link="${name}_steer_link" />
       <origin xyz="${pose_xyz}" rpy="0 0 0" />
-      <axis xyz="0 0 -1" />
+      <axis xyz="0 0 1" />
       <limit lower="${-M_PI/3}" upper="${M_PI/3}" effort="7.0" velocity="2.16"/>
       <dynamics damping="0.0" friction="0.0"/>

File: adrv_description/urdf/wheel.urdf.xacro (robot description, xacro)
@@ -1,4 +1,5 @@
 <?xml version="1.0" ?>
 <robot name="wheel" xmlns:xacro="http://ros.org/wiki/xacro">
+  <xacro:include filename="$(find adrv_description)/urdf/inertia.urdf.xacro" />
   <xacro:macro name="wheel" params="name right_left">
     <link name="${name}_link">
@@ -31,5 +32,6 @@
         </collision>
       </xacro:if>
-      <inertial>
+      <xacro:cylinder_inertia mass="0.3" r="0.016" h="0.03" />
+      <!-- <inertial>
         <origin xyz="0 0 0" />
         <mass value="1.0" />
@@ -37,12 +39,20 @@
                            iyy="1.0" iyz="0.0"
                                      izz="1.0" />
-      </inertial>
+      </inertial> -->
     </link>
     <gazebo reference="${name}_link">
-      <mu1 value="1.0" />
+			<mu1 value="1.0"/>
+			<mu2 value="1.0"/>
+			<kp value="10000000.0" />
+			<kd value="1.0" />
+			<fdir1 value="1 0 0"/>
+      <!-- <mu1 value="1.0" />
       <mu2 value="1.0" />
       <kp  value="100000000.0" />
-      <kd  value="1.0" />
+      <kd  value="100000000.0" />
       <fdir1 value="1 0 0" />
+      <maxVel value="1.0" />
+      <minDepth value="0.005" />
+      <dampingFactor value="0.99" /> -->
     </gazebo>
   </xacro:macro>

File: adrv_description/urdf/ydlidar_x4.urdf.xacro (robot description, xacro)
@@ -31,11 +31,12 @@
     <gazebo reference="${name}_link">
       <sensor type="ray" name="${name}">
+        <!-- <turnGravityOff>true</turnGravityOff> -->
         <pose>0 0 0 0 0 0</pose>
-        <visualize>true</visualize>
+        <visualize>false</visualize>
         <update_rate>12</update_rate>
         <ray>
           <scan>
             <horizontal>
-              <sample>720</sample>
+              <samples>720</samples>
               <resolution>1</resolution>
               <min_angle>0</min_angle>
@@ -57,4 +58,5 @@
           <topicName>scan</topicName>
           <frameName>${name}_link</frameName>
+          <robotNamespace>/</robotNamespace>
         </plugin>
       </sensor>
